File: beba.sch (EAGLE design)
At the start: 37 parts, among them IC1 LT1302SO08, IC2 MCP73871-2AAI/ML

Commit message: - rewrote schematic into sheets
Parts:
- removed C1: 10uF, resistor:C-EUC0805
- removed C2, C3, C5: 10μF, resistor:C-EUC0805
- removed C4, C6: 220μF, resistor:C-EUC1210
- removed C7: 0.1μF, resistor:C-EUC0805
- removed C8: 4700μF / 10V, rcl:CPOL-EUE2,5-6E
- removed CONN1: MX500075-1517USB_MINI-B, MX500075-1517 USB Mini-B straight socket:MX500075-1517USB_MINI-B
- removed CONN2: LiIon, jst-ph:JST-PH2
- removed CONN3: 5VDC, jst-ph:JST-PH2
- removed CONN4: USB-A female socket, right angle, 1734366-1 USB-A socket, vertical:USB-A
- removed D1: BAT60J, diode:BAT60J
- removed D2: MBRS130LT3, diode:MBRS130LT3
- removed IC1: LT1302SO08, adafruit:LT1302SO08
- removed IC2: MCP73871-2AAI/ML, MCP73871 - Powerpath and Charge Controller:MCP73871-2AAI/ML
- removed L1: DJNR6045-100-S, DJNR6045-100S Power Inductor:DJNR6045-100-S
- removed L2: DE1205-18, DE1205-18 Power Inductor:DE1205-18
- removed LED1: green, led:LEDSML1206
- removed LED2: orange, led:LEDSML1206
- removed LED3: red, led:LEDSML1206
- removed R10, R5: 100k, resistor:R-EU_R0805
- removed R11, R13: 75k, resistor:R-EU_R0805
- removed R12, R14: 49k9, resistor:R-EU_R0805
- removed R15: 270k, resistor:R-EU_R0805
- removed R6, R9: 1k, resistor:R-EU_R0805
- removed R7: 150k, resistor:R-EU_R0805
- removed R8: NTC - 10k, resistor:R-EU_0204/5
- removed S1: POWER, smd-special:SWS001
- added CN1, CN2, CN3: S2B-PH-K-S, adafruit:JST_2PIN-THM-RA
- added USB-B1: 67503-1230, MX-67503-1230 USB Mini-B SMT straight socket:MX-67503-1230
- added X1: 62900416021, con-yamaichi:USB-A003
- R1, R3: value 1k -> 75k
- R2: value 1k -> 49k9
- R4: value 270k -> 49k9
Connections:
- removed net 5V0: C2.1, C8.+, D1.A, D1.C, IC2.!TE!, IC2.CE, IC2.IN1, IC2.IN2, IC2.PROG2, IC2.SEL, L1.1
- removed net IT: IC1.IT, R15.1
- removed net N$1: LED3.A, R3.2
- removed net N$10: R6.2, R7.1, R8.1
- removed net N$2: LED2.A, R2.2
- removed net N$3: LED1.A, R1.2
- removed net N$4: D2.A, L2.L1
- removed net PG: IC2.!PG!, LED3.C
- removed net PROG1: IC2.PROG1, R9.1
- removed net PROG3: IC2.PROG3, R10.1
- removed net SHDN: IC1.SHDN, S1.2
- removed net STAT1: IC2.STAT1/!LBO!, LED2.C
- removed net STAT2: IC2.STAT2, LED1.C
- removed net SW: IC1.SW
- removed net THERM: IC2.THERM, R6.1
- removed net VC: C5.2, IC1.VC
- removed net VCC: C4.2, CONN4.VCC, D2.C, IC1.SNS, R11.2, R13.2, R4.2
- removed net VUSB: CONN1.VBUS, CONN3.2, L1.2
- removed net V_LIION_REGULATED: C3.1, C6.2, C7.2, IC1.VIN, IC2.OUT1, IC2.OUT2, L2.L2, R1.1, R2.1, R3.1, S1.1
- new net 5V0_IN: R1.1, R2.1, R3.1, R4.2
- new net 5V0_OUT: R1.2, R3.2, X1.1
- new net LED1_A: R1.2
- new net LED2_A: R2.2
- new net LED3_A: R3.2
- new net VINPUT1: CN1.2
- new net VINPUT2: CN2.2
- new net VUSB_MINI-B: USB-B1.VBUS
- net GND: now also CN1.1, CN2.1, CN3.1, R2.1, R4.1, USB-B1.GND, X1.4; no longer C1.2, C2.2, C3.2, C4.1, C5.1, C6.1, C7.1, C8.-, CONN1.GND, CONN2.2, CONN3.1, CONN4.GND, IC1.GND, IC1.PGND, IC2.GND1, IC2.GND2, IC2.GND3, IC2.GND4, IC2.GND5, IC2.GND6, R10.2, R12.1, R14.1, R15.2, R5.1, R7.2, R8.2, R9.2
- net USBDN: now also R1.1, R2.2, X1.2; no longer CONN4.DN, R11.1, R12.2
- net USBDP: now also R3.1, R4.2, X1.3; no longer CONN4.DP, R13.1, R14.2
- net VPCC: no longer IC2.VPCC, R5.2
- net V_LIION+: now also CN3.2; no longer C1.1, CONN2.1, IC2.VBAT1, IC2.VBAT2, IC2.VBAT_SENSE
Other:
- note added: "Li-Ion Battery"
- note added: "USB downstream facing"
- note added: "USB upstream facing"
- note added: "input #1"
- note added: "input #2"
- moved on the sheet: R1, R2, R3, R4

Commit message: - finalized rev.1 schematic, ERC checks out OK - compiled BOM
Parts:
- removed CN1, CN2, CN3: S2B-PH-K-S, adafruit:JST_2PIN-THM-RA
- removed USB-B1: 67503-1230, MX-67503-1230 USB Mini-B SMT straight socket:MX-67503-1230
- removed X1: 62900416021, con-yamaichi:USB-A003
- added D1: 3SMBJ5921B-TP, diode:ZENER-DIODEDO214AA
- added PAD1: IN2, wirepad:SMD5
- added PAD2, PAD4, PAD7: GND, wirepad:SMD5
- added PAD3: IN3, wirepad:SMD5
- added PAD5: NTC, wirepad:SMD5
- added PAD6: Li-Ion +, wirepad:SMD5
- added USB1: MUSBR-05-F-O-B-SM-A, MUSBR-05-F-O-B-SM-A - Mini USB B Jack:MUSBR-05-F-O-B-SM-A
- added USB2: USB-A-S-S-B-SM2, USB-A-S-S-B-SM2 - USB A Jack:USB-A-S-X-X-SM2
Connections:
- removed net 5V0_IN: R1.1, R2.1, R3.1, R4.2
- removed net 5V0_OUT: R1.2, R3.2, X1.1
- removed net VUSB_MINI-B: USB-B1.VBUS
- new net 5V0: R1.2, R3.2, USB2.VCC
- new net N$8: R1.1
- new net NTC: PAD5.P
- new net VINPUT3: PAD3.P
- new net V_IN: R1.1, R1.2, R2.1, R3.1, R4.2
- new net V_INPUT: D1.C
- net GND: now also D1.A, PAD2.P, PAD4.P, PAD7.P, USB1.GND, USB2.GND; no longer CN1.1, CN2.1, CN3.1, USB-B1.GND, X1.4
- net USBDN: now also USB2.D-; no longer X1.2
- net USBDP: now also USB2.D+; no longer X1.3
- net VINPUT1: now also USB1.VCC; no longer CN1.2
- net VINPUT2: now also PAD1.P; no longer CN2.2
- net V_LIION+: now also PAD6.P; no longer CN3.2
Other:
- note added: "NTC: NXFT15XH103FEAB045"
- note added: "R4"
- note added: "R5"
- note added: "USB-A: upstream facing"
- note added: "Vzener = 6.8V"
- note added: "connect 10k NTC to GND"
- note added: "ds. p. 14: Voltage Proportional Charge Control Vvpcc = ( R5 / (R5+R4) ) * Vin = (100k / (150k))* 5.0V = 3.3V voltages below 3V3 will cause no charging"
- note added: "ds. p. 15 Input Source Type Selection high = share 1.65A between system load and charging"
- note added: "ds. p. 15 USB current regulation set high = 500mA"
- note added: "ds. p. 15, 3.8: fast charge Ireg = 1000V/Rprog1 = 1000/1 = 1000mA"
- note added: "ds. p. 16 Charge Enable high = enabled"
- note added: "ds. p. 16 Timer Enable high = disabled"
- note added: "ds. p. 19, 4.7: charge termination Iterm = 1000V / Rprog3 = 1000V/100 = 10 mA"
- note added: "input #3"
- note added: "max. 7.0V"
- note added: "mini USB-B: downstream facing"
- note added: "schematic according to ds. p. 26, 9.3 - typical application for fixed voltage version"
- note removed: "Li-Ion Battery"
- note removed: "USB downstream facing"
- note removed: "USB upstream facing"
- moved on the sheet: R1, R2, R3, R4

Commit message: - moved over voltage protection diode to forward of ideal diode and duplicated it for the other non-USB input channel - updated BOM
Parts:
- removed D1: 3SMBJ5921B-TP, diode:ZENER-DIODEDO214AA
- removed PAD1: IN2, wirepad:SMD5
- removed PAD2, PAD4: GND, wirepad:SMD5
- removed PAD3: IN3, wirepad:SMD5
- removed R1, R3: 75k, resistor:R-EU_R0805
- removed R2, R4: 49k9, resistor:R-EU_R0805
- added D101, D102: 3SMBJ5921B-TP, diode:ZENER-DIODEDO214AA
- added PAD101: IN2, wirepad:SMD5
- added PAD102, PAD104: GND, wirepad:SMD5
- added PAD103: IN3, wirepad:SMD5
- added R101, R103: 75k, resistor:R-EU_R0805
- added R102, R104: 49k9, resistor:R-EU_R0805
- renumbered PAD5 to PAD105, PAD6 to PAD106, PAD7 to PAD107, USB1 to USB101, USB2 to USB102
Connections:
- removed net LED1_A: R1.2
- removed net LED2_A: R2.2
- removed net LED3_A: R3.2
- removed net N$8: R1.1
- removed net VPCC: R4.1
- removed net V_IN: R1.1, R1.2, R2.1, R3.1, R4.2
- removed net V_INPUT: D1.C
- net 5V0: now also R101.2, R103.2; no longer R1.2, R3.2
- net GND: now also D101.A, D102.A, PAD102.P, PAD104.P, R102.1, R104.1; no longer D1.A, PAD2.P, PAD4.P, R2.1, R4.1
- net USBDN: now also R101.1, R102.2; no longer R1.1, R2.2
- net USBDP: now also R103.1, R104.2; no longer R3.1, R4.2
- net VINPUT2: now also D101.C, PAD101.P; no longer PAD1.P
- net VINPUT3: now also D102.C, PAD103.P; no longer PAD3.P
