File: beba.sch (EAGLE design)
At the start: 15 parts

Commit message: - added fiducials
Parts:
- added FID1, FID2, FID3: (no value), fiducials:FIDUCIALFID_0.5MM
Changed lines of the file:
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@@
 <part name="GND4" library="supply1" library_urn="urn:adsk.eagle:library:371" deviceset="GND" device=""/>
 <part name="GND5" library="supply1" library_urn="urn:adsk.eagle:library:371" deviceset="GND" device=""/>
+<part name="FID1" library="fiducials" deviceset="FIDUCIAL" device="FID_0.5MM"/>
+<part name="FID2" library="fiducials" deviceset="FIDUCIAL" device="FID_0.5MM"/>
+<part name="FID3" library="fiducials" deviceset="FIDUCIAL" device="FID_0.5MM"/>
 </parts>
 <sheets>
@@
 <attribute name="VALUE" x="76.2" y="132.08" size="1.778" layer="96" rot="R270"/>
 </instance>
+<instance part="FID1" gate="G$1" x="78.74" y="83.82" smashed="yes"/>
+<instance part="FID2" gate="G$1" x="78.74" y="73.66" smashed="yes"/>
+<instance part="FID3" gate="G$1" x="78.74" y="63.5" smashed="yes"/>
 </instances>
 <busses>

Commit message: - uploaded brd to fab - created gerber files - rev.1 finished
Parts:
- FID1, FID2, FID3: value (none) -> fiducial
Changed lines of the file:
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@@
 <part name="GND4" library="supply1" library_urn="urn:adsk.eagle:library:371" deviceset="GND" device=""/>
 <part name="GND5" library="supply1" library_urn="urn:adsk.eagle:library:371" deviceset="GND" device=""/>
-<part name="FID1" library="fiducials" deviceset="FIDUCIAL" device="FID_0.5MM"/>
-<part name="FID2" library="fiducials" deviceset="FIDUCIAL" device="FID_0.5MM"/>
-<part name="FID3" library="fiducials" deviceset="FIDUCIAL" device="FID_0.5MM"/>
+<part name="FID1" library="fiducials" deviceset="FIDUCIAL" device="FID_0.5MM" value="fiducial"/>
+<part name="FID2" library="fiducials" deviceset="FIDUCIAL" device="FID_0.5MM" value="fiducial"/>
+<part name="FID3" library="fiducials" deviceset="FIDUCIAL" device="FID_0.5MM" value="fiducial"/>
 </parts>
 <sheets>

Commit message: - optimization of BOM: replaced MCP73871's VPCC 50k resistor with 49.9k
Other:
- note added: "ds. p. 14: Voltage Proportional Charge Control Vvpcc = ( R5 / (R5+R4) ) * Vin = (100k / (149.9k))* 5.0V = 3.36V voltages below 3V3 will cause no charging"
- note removed: "ds. p. 14: Voltage Proportional Charge Control Vvpcc = ( R5 / (R5+R4) ) * Vin = (100k / (150k))* 5.0V = 3.3V voltages below 3V3 will cause no charging"
Changed lines of the file:
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@@
 <sheet>
 <plain>
-<text x="127" y="50.8" size="1.778" layer="97" align="top-left">ds. p. 14: Voltage Proportional Charge Control
-Vvpcc = ( R5 / (R5+R4) ) * Vin
-      = (100k / (150k))* 5.0V
-      = 3.3V
-voltages below 3V3 will cause no charging</text>
 <text x="106.68" y="50.8" size="1.778" layer="97">R4</text>
 <text x="106.68" y="40.64" size="1.778" layer="97">R5</text>
@@
 <wire x1="93.98" y1="101.6" x2="93.98" y2="134.62" width="0.1524" layer="97"/>
 <wire x1="93.98" y1="134.62" x2="99.06" y2="134.62" width="0.1524" layer="97"/>
+<text x="124.46" y="53.34" size="1.778" layer="97" align="top-left">ds. p. 14: Voltage Proportional Charge Control
+Vvpcc = ( R5 / (R5+R4) ) * Vin
+      = (100k / (149.9k))* 5.0V
+      = 3.36V
+voltages below 3V3 will cause no charging</text>
 </plain>
 <instances>

Commit message: start of rev.2 board - increased uninterrupted copper below MCP73871 for better cooling - removed bottom copper contacts for IN1/IN2, GND and similar - replaced MCP73871's big input cap from TH to SMD - replaced NTC solderpads with 0805 component
Parts:
- removed PAD105: NTC, wirepad:SMD5
- added R1: 10k NTC, beta 3892, rcl:R-EU_R0805
Connections:
- new net LED1_A: R1.2
- new net N$8: R1.1
- new net V_IN: R1.1, R1.2
- net GND: now also R1.1
- net NTC: now also R1.2; no longer PAD105.P
Other:
- note removed: "connect 10k NTC to GND"
Changed lines of the file:
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@@
 <part name="GND4" library="supply1" library_urn="urn:adsk.eagle:library:371" deviceset="GND" device=""/>
 <part name="GND5" library="supply1" library_urn="urn:adsk.eagle:library:371" deviceset="GND" device=""/>
-<part name="C16" library="C-Pol" deviceset="C-POL" device="" value="6800uF / 16V"/>
+<part name="C16" library="C-Pol" deviceset="C-POL" device="SMD" value="6800uF / 16V"/>
 <part name="FRAME1" library="frames" library_urn="urn:adsk.eagle:library:229" deviceset="A4L-LOC" device="" value="LiIon charger/powerpath controller"/>
 <part name="C1" library="rcl" library_urn="urn:adsk.eagle:library:334" deviceset="C-EU" device="C0805" package3d_urn="urn:adsk.eagle:package:23617/2" value="10uF / 25V"/>
@@
 <part name="PAD107" library="wirepad" library_urn="urn:adsk.eagle:library:412" deviceset="SMD5" device="" package3d_urn="urn:adsk.eagle:package:30841/1" value="GND"/>
 <part name="PAD106" library="wirepad" library_urn="urn:adsk.eagle:library:412" deviceset="SMD5" device="" package3d_urn="urn:adsk.eagle:package:30841/1" value="Li-Ion +"/>
-<part name="PAD105" library="wirepad" library_urn="urn:adsk.eagle:library:412" deviceset="SMD5" device="" package3d_urn="urn:adsk.eagle:package:30841/1" value="NTC"/>
 <part name="PAD101" library="wirepad" library_urn="urn:adsk.eagle:library:412" deviceset="SMD5" device="" package3d_urn="urn:adsk.eagle:package:30841/1" value="IN2"/>
 <part name="PAD102" library="wirepad" library_urn="urn:adsk.eagle:library:412" deviceset="SMD5" device="" package3d_urn="urn:adsk.eagle:package:30841/1" value="GND"/>
@@
 <part name="FID2" library="fiducials" deviceset="FIDUCIAL" device="FID_0.5MM" value="fiducial"/>
 <part name="FID3" library="fiducials" deviceset="FIDUCIAL" device="FID_0.5MM" value="fiducial"/>
+<part name="R1" library="rcl" library_urn="urn:adsk.eagle:library:334" deviceset="R-EU_" device="R0805" package3d_urn="urn:adsk.eagle:package:23553/2" value="10k NTC, beta 3892"/>
+<part name="GND6" library="supply1" library_urn="urn:adsk.eagle:library:371" deviceset="GND" device=""/>
 </parts>
 <sheets>
@@
 <text x="40.64" y="121.92" size="1.778" layer="97" rot="R180" align="center">input #3</text>
 <text x="38.1" y="165.1" size="1.778" layer="97" rot="R180" align="center">input #1</text>
-<text x="154.94" y="139.7" size="1.778" layer="97">connect
-10k NTC to GND</text>
 <text x="50.8" y="147.32" size="1.778" layer="97">max. 7.0V</text>
 <text x="50.8" y="124.46" size="1.778" layer="97">max. 7.0V</text>
@@
 <attribute name="VALUE" x="154.94" y="132.08" size="1.778" layer="96" rot="R180"/>
 </instance>
-<instance part="PAD105" gate="1" x="157.48" y="137.16" smashed="yes">
-<attribute name="VALUE" x="154.94" y="137.16" size="1.778" layer="96" rot="R180"/>
-</instance>
 <instance part="PAD101" gate="1" x="58.42" y="144.78" smashed="yes">
 <attribute name="NAME" x="55.88" y="144.78" size="1.778" layer="95" rot="R180"/>
@@
 <instance part="FID2" gate="G$1" x="78.74" y="73.66" smashed="yes"/>
 <instance part="FID3" gate="G$1" x="78.74" y="63.5" smashed="yes"/>
+<instance part="R1" gate="G$1" x="167.64" y="137.16" smashed="yes">
+<attribute name="NAME" x="167.64" y="139.7" size="1.778" layer="95"/>
+<attribute name="VALUE" x="165.1" y="139.7" size="1.778" layer="96" align="bottom-right"/>
+</instance>
+<instance part="GND6" gate="1" x="157.48" y="134.62" smashed="yes">
+<attribute name="VALUE" x="154.94" y="134.62" size="1.778" layer="96" rot="R180"/>
+</instance>
 </instances>
 <busses>
@@
 <wire x1="76.2" y1="137.16" x2="76.2" y2="134.62" width="0.1524" layer="91"/>
 <pinref part="GND5" gate="1" pin="GND"/>
+</segment>
+<segment>
+<pinref part="R1" gate="G$1" pin="1"/>
+<wire x1="162.56" y1="137.16" x2="157.48" y2="137.16" width="0.1524" layer="91"/>
+<pinref part="GND6" gate="1" pin="GND"/>
 </segment>
 </net>
@@
 <segment>
 <portref moduleinst="MCP73871-1" port="NTC"/>
-<wire x1="175.26" y1="137.16" x2="160.02" y2="137.16" width="0.1524" layer="91"/>
-<label x="167.64" y="137.16" size="1.778" layer="95"/>
-<pinref part="PAD105" gate="1" pin="P"/>
-</segment>
-</net>
+<wire x1="175.26" y1="137.16" x2="172.72" y2="137.16" width="0.1524" layer="91"/>
+<pinref part="R1" gate="G$1" pin="2"/>
+</segment>
+</net>

Commit message: further work on rev.2 board: - increased copper below MCP73871 even more - replaced solder pads for LiIon battery with SMD JST-PH connector
Parts:
- removed PAD106: Li-Ion +, wirepad:SMD5
- removed PAD107: GND, wirepad:SMD5
- removed R1: 10k NTC, beta 3892, rcl:R-EU_R0805
- added J101: S2B-PH-SM4-TB(LF)(SN), JST-PH:S2B-PH-SM4-TB(LF)(SN)
- added R105: 49k9, resistor:R-EU_R0805
- R101: value 75k -> 10k NTC, beta 3892; device resistor:R-EU_R0805 -> rcl:R-EU_R0805
- R102, R104: value 49k9 -> 75k
- R103: value 75k -> 49k9
- renumbered FID1 to FID101, FID2 to FID102, FID3 to FID103
Connections:
- removed net LED1_A: R1.2
- removed net N$8: R1.1
- removed net V_IN: R1.1, R1.2
- net 5V0: now also R102.2, R104.2; no longer R101.2, R103.2
- net GND: now also J101.2, J101.SHIELD, R101.1, R103.1, R105.1; no longer PAD107.P, R1.1, R102.1, R104.1
- net NTC: now also R101.2; no longer R1.2
- net USBDN: now also R102.1, R103.2; no longer R101.1, R102.2
- net USBDP: now also R104.1, R105.2; no longer R103.1, R104.2
- net V_LIION+: now also J101.1; no longer PAD106.P
Other:
- note removed: "NTC: NXFT15XH103FEAB045"
- moved on the sheet: R101, R102, R103, R104
