File: beba.brd (EAGLE design)
At the start: 77 x 20 mm, 48 parts, among them CN1 S2B-PH-K-S, CN2 S2B-PH-K-S, CN3 S2B-PH-K-S, X1 62900416021

Commit message: - uploaded brd to fab - created gerber files - rev.1 finished
Parts:
- removed CN1, CN2, CN3: S2B-PH-K-S, adafruit:JST-PH-2-THM-RA
- removed IDEAL_DIODE1:C1, IDEAL_DIODE2:C1, IDEAL_DIODE3:C1, TPS630701-1:C11: 0.1μF, rcl:C0805
- removed IDEAL_DIODE1:IC1, IDEAL_DIODE2:IC1, IDEAL_DIODE3:IC1: SIA456DJ-T1-GE3, SIA456DJ-T1-GE3 N-Fet:SC-70-6
- removed IDEAL_DIODE1:IC2, IDEAL_DIODE2:IC2, IDEAL_DIODE3:IC2: LM74670QDGKTQ1, LM74670 - Smart Diode Rectifier Controller:VSSOP-8
- removed MCP73871-1:C16: 4700μF / 10V, C-Pol:TH
- removed MCP73871-1:C4: 10μF, resistor:C0805
- removed MCP73871-1:C6, MCP73871-1:C7: 10u, resistor:C0805
- removed MCP73871-1:IC7: (no value), MCP73871 - Powerpath and Charge Controller:QFN50P400X400X100-21N
- removed MCP73871-1:LED1: LTST-C230KRKT - red, led:SML1206
- removed MCP73871-1:LED2: LTST-C230KGKT - green, led:SML1206
- removed MCP73871-1:LED3: LTST-C230KSKT - yellow, led:SML1206
- removed MCP73871-1:R1, MCP73871-1:R2, MCP73871-1:R3, MCP73871-1:R6, MCP73871-1:R7: 1k, resistor:R0805
- removed MCP73871-1:R10: NTC - 10k, resistor:0204/5
- removed MCP73871-1:R4: 270k, resistor:R0805
- removed MCP73871-1:R5, MCP73871-1:R8: 100k, resistor:R0805
- removed MCP73871-1:R9: 150k, resistor:R0805
- removed R1, R3: 75k, resistor:R0805
- removed R2, R4: 49k9, resistor:R0805
- removed TPS630701-1:C10, TPS630701-1:C12, TPS630701-1:C8, TPS630701-1:C9: 10u, rcl:C0805
- removed TPS630701-1:C13, TPS630701-1:C14, TPS630701-1:C15: 22u, rcl:C0805
- removed TPS630701-1:IC8: TPS630701, TPS630701 - Buck Boost 5V regulator:VQFN
- removed TPS630701-1:L1: XFL4020-152MEB, XFL4020-152MEC Inductor 1.5uH:SMD
- removed TPS630701-1:R11: 100k, rcl:R0805
- removed TPS630701-1:R12: 10k, rcl:R0805
- removed USB-B1: 67503-1230, MX-67503-1230 USB Mini-B SMT straight socket:SMT
- removed X1: 62900416021, con-yamaichi:USB-A003
- added C201, C301, C401, C611: 0.1uF / 50V, rcl:C0805
- added C501, C502, C503, C608, C609, C610, C612: 10uF / 6.3V, rcl:C0805
- added C516: 4700uF / 10V, C-Pol:TH
- added C613, C614, C615: 22u / 10V, rcl:C0805
- added D101, D102: 3SMBJ5921B-TP, diode:DO214AA
- added FID1, FID2, FID3: fiducial, fiducials:FIDUCIAL_0.5MM
- added IC202, IC302, IC402: LM74670QDGKTQ1, LM74670 - Smart Diode Rectifier Controller:VSSOP-8
- added IC507: 579-MCP73871T2CCIML, MCP73871 - Powerpath and Charge Controller:QFN50P400X400X100-21N
- added IC601: TPS630701RNMT, TPS630701 - Buck Boost 5V regulator:VQFN
- added L602: XFL4020-152MEC, XFL4020 - Inductor:1616
- added LED501: LTST-C230KRKT - red, led:SML1206
- added LED502: LTST-C230KGKT - green, led:SML1206
- added LED503: LTST-C230KSKT - yellow, led:SML1206
- added PAD101: IN2, wirepad:SMD2,54-5,08
- added PAD102, PAD104, PAD107: GND, wirepad:SMD2,54-5,08
- added PAD103: IN3, wirepad:SMD2,54-5,08
- added PAD105: NTC, wirepad:SMD2,54-5,08
- added PAD106: Li-Ion +, wirepad:SMD2,54-5,08
- added Q202, Q302, Q402: SQ2310ES-T1_BE3, transistor-small-signal:SOT23
- added R101, R103: 75k, resistor:R0805
- added R102, R104: 49k9, resistor:R0805
- added R501, R502, R503, R506, R507: 1k, resistor:R0805
- added R504: 50k, resistor:R0805
- added R505, R508, R606: 100k, resistor:R0805
- added R509: 150k, resistor:R0805
- added R601: 10k, resistor:R0805
- added USB101: MUSBR-05-F-O-B-SM-A, MUSBR-05-F-O-B-SM-A - Mini USB B Jack:SAMTEC_MUSBR-05-F-O-B-SM-A
- added USB102: USB-A-S-S-B-SM2, USB-A-S-S-B-SM2 - USB A Jack:SAMTEC_USB-A-S-X-X-SM2
Connections:
- removed net 5V0_IN: IDEAL_DIODE1:IC1.1_D, IDEAL_DIODE1:IC1.2_D, IDEAL_DIODE1:IC1.5_D, IDEAL_DIODE1:IC1.6_D, IDEAL_DIODE1:IC1.8_D, IDEAL_DIODE1:IC2.CATHODE, IDEAL_DIODE2:IC1.1_D, IDEAL_DIODE2:IC1.2_D, IDEAL_DIODE2:IC1.5_D, IDEAL_DIODE2:IC1.6_D, IDEAL_DIODE2:IC1.8_D, IDEAL_DIODE2:IC2.CATHODE, IDEAL_DIODE3:IC1.1_D, IDEAL_DIODE3:IC1.2_D, IDEAL_DIODE3:IC1.5_D, IDEAL_DIODE3:IC1.6_D, IDEAL_DIODE3:IC1.8_D, IDEAL_DIODE3:IC2.CATHODE
- removed net 5V0_OUT: R1.2, R3.2, X1.1
- removed net MCP73871-1:5V0_IN: MCP73871-1:C16.POS, MCP73871-1:C4.1, MCP73871-1:IC7.17_CE, MCP73871-1:IC7.18_IN1, MCP73871-1:IC7.19_IN2, MCP73871-1:IC7.3_SEL, MCP73871-1:IC7.4_PROG2, MCP73871-1:IC7.9_!TE!, MCP73871-1:R1.1, MCP73871-1:R2.1, MCP73871-1:R3.1, MCP73871-1:R4.2
- removed net MCP73871-1:N$10: MCP73871-1:R10.1, MCP73871-1:R6.2, MCP73871-1:R9.1
- removed net MCP73871-1:V_LIION+: MCP73871-1:C7.1, MCP73871-1:IC7.14_VBAT1, MCP73871-1:IC7.15_VBAT2, MCP73871-1:IC7.16_BAT_SENSE
- removed net MCP73871-1:V_LIION_REGULATED: MCP73871-1:C6.1, MCP73871-1:IC7.1_OUT1, MCP73871-1:IC7.20_OUT2
- removed net TPS630701-1:5V0_OUT: TPS630701-1:C12.2, TPS630701-1:C13.2, TPS630701-1:C14.2, TPS630701-1:C15.2, TPS630701-1:IC8.5-FB, TPS630701-1:IC8.7-VOUT, TPS630701-1:IC8.8-VOUT, TPS630701-1:IC8.VOUT, TPS630701-1:R11.2
- removed net VUSB_MINI-B: IDEAL_DIODE1:IC1.4_S, IDEAL_DIODE1:IC1.7_S, IDEAL_DIODE1:IC2.ANODE, USB-B1.VBUS
- removed net V_LIION_REGULATED: TPS630701-1:C10.2, TPS630701-1:C8.2, TPS630701-1:C9.2, TPS630701-1:IC8.12-VIN, TPS630701-1:IC8.13-VIN, TPS630701-1:IC8.VIN, TPS630701-1:R12.2
- new net 5V0: C612.2, C613.2, C614.2, C615.2, IC601.5-FB, IC601.7-VOUT, IC601.8-VOUT, IC601.VOUT, R101.2, R103.2, R606.2, USB102.1_5V0
- new net NTC: PAD105.1, R506.2, R509.1
- new net VINPUT3: D102.C, IC402.ANODE, PAD103.1, Q402.2
- new net V_INPUT: C503.1, C516.POS, IC202.CATHODE, IC302.CATHODE, IC402.CATHODE, IC507.17_CE, IC507.18_IN1, IC507.19_IN2, IC507.3_SEL, IC507.4_PROG2, IC507.9_!TE!, Q202.3, Q302.3, Q402.3, R501.1, R502.1, R503.1, R504.2
- new net V_REGULATED: C502.1, C608.2, C609.2, C610.2, IC507.1_OUT1, IC507.20_OUT2, IC601.12-VIN, IC601.13-VIN, IC601.VIN, R601.2
- net GND: now also C501.2, C502.2, C503.2, C516.NEG, C608.1, C609.1, C610.1, C611.1, C612.1, C613.1, C614.1, C615.1, D101.A, D102.A, IC507.10_GND1, IC507.11_GND2, IC507.GND2, IC507.GND3, IC507.GND4, IC507.GND5, IC507.GND6, IC601.10-PGND, IC601.15-VSEL, IC601.4-GND, IC601.6-FB2, PAD102.1, PAD104.1, PAD107.1, R102.1, R104.1, R505.1, R507.2, R508.2, R509.2, USB101.5_GND, USB101.G1, USB101.G2, USB101.G3, USB101.G4, USB102.4_GND, USB102.G1, USB102.G2; no longer CN1.2, CN2.2, CN3.2, MCP73871-1:C16.NEG, MCP73871-1:C4.2, MCP73871-1:C6.2, MCP73871-1:C7.2, MCP73871-1:IC7.10_GND1, MCP73871-1:IC7.11_GND2, MCP73871-1:IC7.GND2, MCP73871-1:IC7.GND3, MCP73871-1:IC7.GND4, MCP73871-1:IC7.GND5, MCP73871-1:IC7.GND6, MCP73871-1:R10.2, MCP73871-1:R5.1, MCP73871-1:R7.2, MCP73871-1:R8.2, MCP73871-1:R9.2, R2.1, R4.1, TPS630701-1:C10.1, TPS630701-1:C11.1, TPS630701-1:C12.1, TPS630701-1:C13.1, TPS630701-1:C14.1, TPS630701-1:C15.1, TPS630701-1:C8.1, TPS630701-1:C9.1, TPS630701-1:IC8.10-PGND, TPS630701-1:IC8.15-VSEL, TPS630701-1:IC8.4-GND, TPS630701-1:IC8.6-FB2, USB-B1.GND1, USB-B1.GND2, USB-B1.GND3, USB-B1.GND4, USB-B1.GND5, X1.4
- net IDEAL_DIODE1:GATE_DRIVER: now also IC202.GATE_DRIVE, IC202.GATE_PULLD, Q202.1; no longer IDEAL_DIODE1:IC1.3_G, IDEAL_DIODE1:IC2.GATE_DRIVE, IDEAL_DIODE1:IC2.GATE_PULLD
- net IDEAL_DIODE1:VCAPH: now also C201.2, IC202.VCAPH; no longer IDEAL_DIODE1:C1.2, IDEAL_DIODE1:IC2.VCAPH
- net IDEAL_DIODE1:VCAPL: now also C201.1, IC202.VCAPL; no longer IDEAL_DIODE1:C1.1, IDEAL_DIODE1:IC2.VCAPL
- net IDEAL_DIODE2:GATE_DRIVER: now also IC302.GATE_DRIVE, IC302.GATE_PULLD, Q302.1; no longer IDEAL_DIODE2:IC1.3_G, IDEAL_DIODE2:IC2.GATE_DRIVE, IDEAL_DIODE2:IC2.GATE_PULLD
- net IDEAL_DIODE2:VCAPH: now also C301.2, IC302.VCAPH; no longer IDEAL_DIODE2:C1.2, IDEAL_DIODE2:IC2.VCAPH
- net IDEAL_DIODE2:VCAPL: now also C301.1, IC302.VCAPL; no longer IDEAL_DIODE2:C1.1, IDEAL_DIODE2:IC2.VCAPL
- net IDEAL_DIODE3:GATE_DRIVER: now also IC402.GATE_DRIVE, IC402.GATE_PULLD, Q402.1; no longer IDEAL_DIODE3:IC1.3_G, IDEAL_DIODE3:IC2.GATE_DRIVE, IDEAL_DIODE3:IC2.GATE_PULLD
- net IDEAL_DIODE3:VCAPH: now also C401.2, IC402.VCAPH; no longer IDEAL_DIODE3:C1.2, IDEAL_DIODE3:IC2.VCAPH
- net IDEAL_DIODE3:VCAPL: now also C401.1, IC402.VCAPL; no longer IDEAL_DIODE3:C1.1, IDEAL_DIODE3:IC2.VCAPL
- net MCP73871-1:LED1_A: now also LED501.A, R501.2; no longer MCP73871-1:LED1.A, MCP73871-1:R1.2
- net MCP73871-1:LED2_A: now also LED502.A, R502.2; no longer MCP73871-1:LED2.A, MCP73871-1:R2.2
- net MCP73871-1:LED3_A: now also LED503.A, R503.2; no longer MCP73871-1:LED3.A, MCP73871-1:R3.2
- net MCP73871-1:PG: now also IC507.!6_PG!, LED501.C; no longer MCP73871-1:IC7.!6_PG!, MCP73871-1:LED1.C
- net MCP73871-1:PROG1: now also IC507.13_PROG1, R507.1; no longer MCP73871-1:IC7.13_PROG1, MCP73871-1:R7.1
- net MCP73871-1:PROG3: now also IC507.12_PROG3, R508.1; no longer MCP73871-1:IC7.12_PROG3, MCP73871-1:R8.1
- net MCP73871-1:STAT1: now also IC507.8_STAT1/!LBO!, LED503.C; no longer MCP73871-1:IC7.8_STAT1/!LBO!, MCP73871-1:LED3.C
- net MCP73871-1:STAT2: now also IC507.7_STAT2, LED502.C; no longer MCP73871-1:IC7.7_STAT2, MCP73871-1:LED2.C
- net MCP73871-1:THERM: now also IC507.5_THERM, R506.1; no longer MCP73871-1:IC7.5_THERM, MCP73871-1:R6.1
- net MCP73871-1:VPCC: now also IC507.2_VPCC, R504.1, R505.2; no longer MCP73871-1:IC7.2_VPCC, MCP73871-1:R4.1, MCP73871-1:R5.2
- net TPS630701-1:L1: now also IC601.11-L1, L602.P$1; no longer TPS630701-1:IC8.11-L1, TPS630701-1:L1.P$1
- net TPS630701-1:L2: now also IC601.9-L2, L602.P$2; no longer TPS630701-1:IC8.9-L2, TPS630701-1:L1.P$2
- net TPS630701-1:N$8: now also IC601.1-PS/S, IC601.14-EN, R601.1; no longer TPS630701-1:IC8.1-PS/S, TPS630701-1:IC8.14-EN, TPS630701-1:R12.1
- net TPS630701-1:PG1: now also IC601.2-PG, R606.1; no longer TPS630701-1:IC8.2-PG, TPS630701-1:R11.1
- net TPS630701-1:VAUX: now also C611.2, IC601.3-VAUX; no longer TPS630701-1:C11.2, TPS630701-1:IC8.3-VAUX
- net USBDN: now also R101.1, R102.2, USB102.2_DN; no longer R1.1, R2.2, X1.2
- net USBDP: now also R103.1, R104.2, USB102.3_DP; no longer R3.1, R4.2, X1.3
- net VINPUT1: now also IC202.ANODE, Q202.2, USB101.1_VCC; no longer CN1.1, IDEAL_DIODE2:IC1.4_S, IDEAL_DIODE2:IC1.7_S, IDEAL_DIODE2:IC2.ANODE
- net VINPUT2: now also D101.C, IC302.ANODE, PAD101.1, Q302.2; no longer CN2.1, IDEAL_DIODE3:IC1.4_S, IDEAL_DIODE3:IC1.7_S, IDEAL_DIODE3:IC2.ANODE
- net V_LIION+: now also C501.1, IC507.14_VBAT1, IC507.15_VBAT2, IC507.16_BAT_SENSE, PAD106.1; no longer CN3.1
Routing:
- net V_INPUT: track 0.00 -> 106.0 mm, vias 0 -> 3
- net MCP73871-1:PG: track 0.00 -> 45.1 mm, vias 0 -> 2
- net MCP73871-1:STAT2: track 0.00 -> 39.4 mm, vias 0 -> 2
- net MCP73871-1:STAT1: track 0.00 -> 34.9 mm, vias 0 -> 2
- net V_REGULATED: track 0.00 -> 17.8 mm, vias 0 -> 6
- net 5V0: track 0.00 -> 16.0 mm, vias 0 -> 8
- net NTC: track 0.00 -> 13.8 mm, vias 0 -> 7
- net VINPUT3: track 0.00 -> 13.3 mm, vias 0 -> 7
- net TPS630701-1:N$8: track 0.00 -> 11.0 mm, vias 0 -> 2
- net TPS630701-1:PG1: track 0.00 -> 10.0 mm, vias 0 -> 2
- net MCP73871-1:PROG1: track 0.00 -> 8.31 mm
- net TPS630701-1:VAUX: track 0.00 -> 8.16 mm, vias 0 -> 2
- net IDEAL_DIODE1:GATE_DRIVER: track 0.00 -> 7.56 mm
- net IDEAL_DIODE3:GATE_DRIVER: track 0.00 -> 7.53 mm
- net IDEAL_DIODE2:GATE_DRIVER: track 0.00 -> 7.53 mm
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- added copper zone on layer 1, net 5V0
- added copper zone on layer 16, net 5V0
- added copper zone on layer 16, net NTC
- added copper zone on layer 1, net TPS630701-1:L1
- added copper zone on layer 1, net TPS630701-1:L2
- added copper zone on layer 1, net VINPUT1
- added copper zone on layer 1, net VINPUT2
- added copper zone on layer 16, net VINPUT2
- added copper zone on layer 1, net VINPUT3
- added copper zone on layer 16, net VINPUT3
- added copper zone on layer 1, net V_INPUT
- added copper zone on layer 16, net V_INPUT
- added copper zone on layer 16, net V_LIION+
- added copper zone on layer 1, net V_REGULATED
- added copper zone on layer 16, net V_REGULATED
- removed copper zone on layer 1, net 5V0_IN
- removed copper zone on layer 1, net 5V0_OUT
- removed copper zone on layer 16, net 5V0_OUT
- removed copper zone on layer 1, net L1
- removed copper zone on layer 1, net L2
- removed copper zone on layer 1, net V_LIION_REGULATED
- removed copper zone on layer 16, net V_LIION_REGULATED
Other:
- board size 77 x 20 mm -> 35 x 56 mm
- board text added: "1s1p Li-Ion only"
- board text added: "GND"
- board text added: "IN2"
- board text added: "IN3"
- board text added: "Li+"
- board text added: "NTC"
- board text added: "PG"
- board text added: "STAT1"
- board text added: "STAT2"
- board text added: "beba rev.1"
- board text added: "charging complete"
- board text added: "charging in progress"
- board text added: "downstream"
- board text added: "ejovrh"
- board text added: "max. 7VDC, 1A"
- board text added: "power good"
- board text added: "upstream"

Commit message: - changed positions of red and green led
Parts:
- LED501: value LTST-C230KRKT - red -> LTST-C230KGKT - green
- LED502: value LTST-C230KGKT - green -> LTST-C230KRKT - red
Changed lines of the file:
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@@
 <attribute name="VALUE" x="-35" y="170" size="1" layer="27" font="vector" rot="R90" align="center"/>
 </element>
-<element name="LED501" library="led" library_urn="urn:adsk.eagle:library:259" package="SML1206" package3d_urn="urn:adsk.eagle:package:15829/1" value="LTST-C230KRKT - red" x="-55" y="130" smashed="yes" rot="R270" grouprefs="LED_PG">
+<element name="LED501" library="led" library_urn="urn:adsk.eagle:library:259" package="SML1206" package3d_urn="urn:adsk.eagle:package:15829/1" value="LTST-C230KGKT - green" x="-55" y="130" smashed="yes" rot="R270" grouprefs="LED_PG">
 <attribute name="NAME" x="-51.5" y="130" size="0.75" layer="25" font="vector" rot="R90" align="center"/>
 <attribute name="POPULARITY" value="6" x="-55" y="130" size="1.778" layer="27" rot="R270" display="off"/>
 <attribute name="VALUE" x="-55" y="130" size="1.27" layer="27" rot="R270"/>
 </element>
-<element name="LED502" library="led" library_urn="urn:adsk.eagle:library:259" package="SML1206" package3d_urn="urn:adsk.eagle:package:15829/1" value="LTST-C230KGKT - green" x="-55" y="136" smashed="yes" rot="R270" grouprefs="LED_STAT2">
+<element name="LED502" library="led" library_urn="urn:adsk.eagle:library:259" package="SML1206" package3d_urn="urn:adsk.eagle:package:15829/1" value="LTST-C230KRKT - red" x="-55" y="136" smashed="yes" rot="R270" grouprefs="LED_STAT2">
 <attribute name="NAME" x="-51.5" y="136" size="0.75" layer="25" font="vector" rot="R90" align="center"/>
 <attribute name="POPULARITY" value="6" x="-55" y="136" size="1.778" layer="27" rot="R270" display="off"/>

Commit message: - exchanged passives (capacitors with higher voltage, resistors with higher power rating), updated BOM
Parts:
- C201, C301, C401: value 0.1uF / 50V -> 0.1uF / 25V
- C501, C502, C503, C608, C609, C610, C612: value 10uF / 6.3V -> 10uF / 25V
- C516: value 4700uF / 10V -> 6800uF / 16V
- C613, C614, C615: value 22u / 10V -> 22u / 25V
